File: Hardware/APRN-pi_board/APRN-pi.kicad_sch (KiCad schematic)
At the start: 34 parts, among them J1 Raspberry_Pi_2_3, J2 Conn_Coaxial, J3 Amplifier Jumper, J4 Screw_Terminal_01x02, J5 AudioJack4, J6 Conn_01x04, Q1 MMBT3906, Q2 MMBT3906, U1 DRA818V, U2 L7805

Commit message: more logos
Parts:
- added L2: KITSUNE_LOGO, KenwoodFox:KITSUNE_LOGO, symbol KenwoodFox:KITSUNE_LOGO
Changed lines of the file:
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@@
     (pin "4")
+  )
+  (symbol (lib_id "Graphic:Logo_Open_Hardware_Small") (at 278.13 172.72 0) (unit 1)
+    (in_bom yes) (on_board yes) (fields_autoplaced)
+    (property "Reference" "#LOGO1" (id 0) (at 278.13 165.735 0)
+      (effects (font (size 1.27 1.27)) hide)
+    )
+    (property "Value" "Logo_Open_Hardware_Small" (id 1) (at 278.13 178.435 0)
+      (effects (font (size 1.27 1.27)) hide)
+    )
+    (property "Footprint" "" (id 2) (at 278.13 172.72 0)
+      (effects (font (size 1.27 1.27)) hide)
+    )
+    (property "Datasheet" "~" (id 3) (at 278.13 172.72 0)
+      (effects (font (size 1.27 1.27)) hide)
+    )
+  )
+  (symbol (lib_id "KenwoodFox:KITSUNE_LOGO") (at 13.97 173.99 0) (unit 1)
+    (in_bom yes) (on_board yes) (fields_autoplaced)
+    (property "Reference" "L2" (id 0) (at 15.24 172.7199 0)
+      (effects (font (size 1.27 1.27)) (justify left))
+    )
+    (property "Value" "KITSUNE_LOGO" (id 1) (at 15.24 175.2599 0)
+      (effects (font (size 1.27 1.27)) (justify left))
+    )
+    (property "Footprint" "KenwoodFox:KITSUNE_LOGO" (id 2) (at 13.97 173.99 0)
+      (effects (font (size 1.27 1.27)) hide)
+    )
+    (property "Datasheet" "" (id 3) (at 13.97 173.99 0)
+      (effects (font (size 1.27 1.27)) hide)
+    )
   )
   (symbol (lib_id "power:GND") (at 160.02 142.24 0) (unit 1)
@@
     )
   )
-  (symbol (lib_id "KenwoodFox:KITSUNE_LOGO") (at 13.97 176.53 0) (unit 1)
-    (in_bom yes) (on_board yes) (fields_autoplaced)
-    (property "Reference" "L1" (id 0) (at 15.24 175.2599 0)
-      (effects (font (size 1.27 1.27)) (justify left))
-    )
-    (property "Value" "KITSUNE_LOGO" (id 1) (at 15.24 177.7999 0)
-      (effects (font (size 1.27 1.27)) (justify left))
-    )
-    (property "Footprint" "KenwoodFox:KITSUNE_LOGO" (id 2) (at 13.97 176.53 0)
-      (effects (font (size 1.27 1.27)) hide)
-    )
-    (property "Datasheet" "" (id 3) (at 13.97 176.53 0)
+  (symbol (lib_id "KenwoodFox:KITSUNE_LOGO") (at 13.97 168.91 0) (unit 1)
+    (in_bom yes) (on_board yes)
+    (property "Reference" "L1" (id 0) (at 15.24 167.6399 0)
+      (effects (font (size 1.27 1.27)) (justify left))
+    )
+    (property "Value" "KITSUNE_LOGO" (id 1) (at 15.24 170.1799 0)
+      (effects (font (size 1.27 1.27)) (justify left))
+    )
+    (property "Footprint" "KenwoodFox:KITSUNE_LOGO" (id 2) (at 13.97 168.91 0)
+      (effects (font (size 1.27 1.27)) hide)
+    )
+    (property "Datasheet" "" (id 3) (at 13.97 168.91 0)
       (effects (font (size 1.27 1.27)) hide)
     )
@@
   )
   (symbol_instances
+    (path "/0d7bc4ee-8b1c-4141-a30f-88ee74c2638f"
+      (reference "#LOGO1") (unit 1) (value "Logo_Open_Hardware_Small") (footprint "")
+    )
     (path "/7a4a7cd3-b322-4799-bd04-d77279f4cccb"
       (reference "#PWR01") (unit 1) (value "GND") (footprint "")
@@
       (reference "L1") (unit 1) (value "KITSUNE_LOGO") (footprint "KenwoodFox:KITSUNE_LOGO")
     )
+    (path "/0d7c7502-6413-4cdb-b85d-145565614a49"
+      (reference "L2") (unit 1) (value "KITSUNE_LOGO") (footprint "KenwoodFox:KITSUNE_LOGO")
+    )
     (path "/d652480f-0bca-4130-8930-ba734e86fe77"

Commit message: Use upstream
Connections:
- net SCL: now also J6.2 (Pin_2); no longer J6.3 (Pin_3)
- net SDA: now also J6.3 (Pin_3); no longer J6.2 (Pin_2)
Changed lines of the file:
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@@
-    (stroke (width 0) (type default) (color 0 0 0 0))
-  )
-  (wire (pts (xy 31.75 154.94) (xy 35.56 154.94))
     (stroke (width 0) (type default) (color 0 0 0 0))
   )
@@
     (stroke (width 0) (type default) (color 0 0 0 0))
   )
-  (wire (pts (xy 31.75 152.4) (xy 35.56 152.4))
-    (stroke (width 0) (type default) (color 0 0 0 0))
-  )
   (wire (pts (xy 242.57 31.75) (xy 257.81 31.75))
     (stroke (width 0) (type default) (color 0 0 0 0))
@@
     (stroke (width 0) (type default) (color 0 0 0 0))
   )
+  (wire (pts (xy 31.75 152.4) (xy 38.1 152.4))
+    (stroke (width 0) (type default) (color 0 0 0 0))
+  )
   (wire (pts (xy 31.75 149.86) (xy 35.56 149.86))
     (stroke (width 0) (type default) (color 0 0 0 0))
@@
   )
   (wire (pts (xy 139.7 139.7) (xy 147.32 139.7))
+    (stroke (width 0) (type default) (color 0 0 0 0))
+  )
+  (wire (pts (xy 31.75 154.94) (xy 38.1 154.94))
     (stroke (width 0) (type default) (color 0 0 0 0))
   )
@@
     )
   )
-  (global_label "SDA" (shape bidirectional) (at 35.56 154.94 0) (fields_autoplaced)
+  (global_label "SDA" (shape bidirectional) (at 38.1 152.4 0) (fields_autoplaced)
     (effects (font (size 1.27 1.27)) (justify left))
-    (property "Intersheet References" "${INTERSHEET_REFS}" (id 0) (at 41.5412 154.8606 0)
+    (property "Intersheet References" "${INTERSHEET_REFS}" (id 0) (at 44.0812 152.3206 0)
       (effects (font (size 1.27 1.27)) (justify left) hide)
     )
@@
     )
   )
-  (global_label "SCL" (shape input) (at 35.56 152.4 0) (fields_autoplaced)
+  (global_label "SCL" (shape input) (at 38.1 154.94 0) (fields_autoplaced)
     (effects (font (size 1.27 1.27)) (justify left))
-    (property "Intersheet References" "${INTERSHEET_REFS}" (id 0) (at 41.4807 152.3206 0)
+    (property "Intersheet References" "${INTERSHEET_REFS}" (id 0) (at 44.0207 154.8606 0)
       (effects (font (size 1.27 1.27)) (justify left) hide)
     )
